Commit message: Enforce limits in hardware interface and controller from urdf limits.

File: src/turret_description/urdf/turret.urdf (robot description, URDF)
Before this commit: robot turret, 4 links, 3 joints
Joints:
- joint pan_joint: limit lower=0.0 upper=180.0 effort=1.0 velocity=45.0 -> lower=0.0 upper=180.0 effort=0.0 velocity=0.0
- joint tilt_joint: limit lower=60.0 upper=120.0 effort=1.0 velocity=45.0 -> lower=90.0 upper=120.0 effort=0.0 velocity=0.0
- joint trigger_joint: limit lower=0.0 upper=180.0 effort=1.0 velocity=45.0 -> lower=0.0 upper=1.0 effort=0.0 velocity=0.0; type revolute -> prismatic

Commit message: Fix pwm width, left joystick y defaults to min angle, only controls when the joystick is moved up

File: src/turret_description/urdf/turret.urdf (robot description, URDF)
Before this commit: robot turret, 4 links, 3 joints
Joints:
- joint tilt_joint: limit lower=90.0 upper=120.0 effort=0.0 velocity=0.0 -> lower=90.0 upper=140.0 effort=0.0 velocity=0.0
